Commit message: refine the sim models

File: rotors_description/urdf/m100.xacro (robot description, xacro)
@@ -21,8 +21,8 @@
   <xacro:property name="rotor_velocity_slowdown_sim" value="10" />
   <xacro:property name="use_mesh_file" value="true" />
-  <xacro:property name="mesh_file" value="package://rotors_description/meshes/m100.dae" />
+  <xacro:property name="mesh_file" value="package://rotors_description/meshes/m100/m100.dae" />
   <xacro:property name="mass" value="2.7" /> <!-- [kg] not included VLP and Cam mount-->
-  <xacro:property name="body_width" value="0.82" /> <!-- [m] -->
-  <xacro:property name="body_height" value="0.22" /> <!-- [m] -->
+  <xacro:property name="body_width" value="0.82" />
+  <xacro:property name="body_height" value="0.22" />
   <xacro:property name="mass_rotor" value="0.106" /> <!-- [kg] -->
   <xacro:property name="arm_length" value="0.32" /> <!-- [m] -->

File: rotors_description/urdf/m100_pccase.xacro (robot description, xacro)
@@ -1,5 +1,5 @@
 <?xml version="1.0"?>
 <robot xmlns:xacro="http://www.ros.org/wiki/xacro">
-	<!-- Macro to add a camera. -->
+	<!-- Macro to add a pc case. -->
   <xacro:macro name="pccase_macro"
     params="namespace parent_link *origin">
