Commit message: refine the sim models

File: rotors_description/urdf/elios_base.xacro (robot description, xacro)
@@ -38,11 +38,4 @@
     <xacro:bag_plugin_macro namespace="${namespace}" bag_file="$(arg log_file)" rotor_velocity_slowdown_sim="${rotor_velocity_slowdown_sim}" wait_to_record_bag="$(arg wait_to_record_bag)" />
   </xacro:if>
-  <!-- VLP16 -->
-  <!-- <xacro:arg name="gpu" default="false"/>
-  <xacro:property name="gpu" value="$(arg gpu)" />
-  <xacro:include filename="$(find velodyne_description)/urdf/VLP-16.urdf.xacro"/>
-  <VLP-16 parent="${namespace}/base_link" name="/velodyne" topic="/velodyne_points" hz="10" samples="440" gpu="${gpu}">
-    <origin xyz="0 0 0.04" rpy="0 0 0" />
-  </VLP-16> -->
   <!-- Os1-64 -->
   <xacro:include filename="$(find lidar_description)/urdf/OS1-64.urdf.xacro"/>

File: rotors_description/urdf/m100_base.xacro (robot description, xacro)
@@ -50,5 +50,5 @@
   <xacro:arg name="gpu" default="false"/>
   <xacro:property name="gpu" value="$(arg gpu)" />
-  <xacro:include filename="$(find velodyne_description)/urdf/VLP-16.urdf.xacro"/>
+  <xacro:include filename="$(find lidar_description)/urdf/VLP-16.urdf.xacro"/>
   <VLP-16 parent="${namespace}/base_link" name="${namespace}/velodyne" topic="/velodyne_points" hz="10" samples="440" gpu="${gpu}">
     <origin xyz="0 0 0.04" rpy="0 0 0" />
