Commit message: Fix acc controller for elios model, add option to use VLP16 or OS1-64

File: rotors_description/urdf/elios.xacro (robot description, xacro)
@@ -16,28 +16,34 @@
   limitations under the License.
 -->
-<robot name="elios" xmlns:xacro="http://ros.org/wiki/xacro">
+<robot name="delta" xmlns:xacro="http://ros.org/wiki/xacro">
   <!-- Properties -->
   <xacro:property name="namespace" value="$(arg namespace)" />
-  <xacro:property name="rotor_velocity_slowdown_sim" value="2" />
+  <xacro:property name="rotor_velocity_slowdown_sim" value="10" />
   <xacro:property name="use_mesh_file" value="true" />
   <xacro:property name="mesh_file" value="package://rotors_description/meshes/elios/elios.dae" />
-  <xacro:property name="mass" value="2.4" /> <!-- [kg] -->
-  <xacro:property name="body_width" value="0.5" /> <!-- [m] -->
-  <xacro:property name="body_height" value="0.5" /> <!-- [m] -->
-  <xacro:property name="mass_rotor" value="0.106" /> <!-- [kg] -->
+  <xacro:property name="mass" value="2.4" /> <!-- [kg] not included VLP and Cam mount-->
+  <xacro:property name="body_width" value="0.5" />
+  <xacro:property name="body_height" value="0.5" />
+  <xacro:property name="mass_rotor" value="0.003" /> <!-- [kg] -->
   <xacro:property name="arm_length" value="0.155" /> <!-- [m] -->
+  <!-- <xacro:property name="mass_arm" value="0.01" /> [kg] -->
   <xacro:property name="rotor_offset_top" value="-0.021" /> <!-- 0.025 [m] -->
-  <xacro:property name="radius_rotor" value="0.0662" /> <!-- [m] -->
-  <xacro:property name="motor_constant" value="0.02246" /> <!-- [kg m/s^2] -->
+  <xacro:property name="radius_rotor" value="0.053" /> <!-- [m] -->
+  <!-- <xacro:property name="motor_constant" value="0.02246" /> --> <!--[kg m/s^2] -->
+  <xacro:property name="motor_constant" value="8.54858e-05" /> <!-- [kg m/s^2] -->
   <xacro:property name="moment_constant" value="0.016" /> <!-- [m] N/A -->
   <xacro:property name="time_constant_up" value="0.0125" /> <!-- [s] N/A -->
-  <xacro:property name="time_constant_down" value="0.1" /> <!-- [s] N/A -->
-  <xacro:property name="max_rot_velocity" value="916.0" /> <!-- [rad/s] -->
+  <xacro:property name="time_constant_down" value="0.025" /> <!-- [s] N/A -->
+  <xacro:property name="max_rot_velocity" value="2000.0" /> <!-- [rad/s] -->
+  <xacro:property name="sin30" value="0.5" />
+  <xacro:property name="cos30" value="0.866025403784" />
 	<xacro:property name="sqrt2inv" value="0.70710678118" />
+  <xacro:property name="sqrt2" value="1.4142135623730951" />
   <xacro:property name="rotor_drag_coefficient" value="8.06428e-05" /> <!-- N/A -->
   <xacro:property name="rolling_moment_coefficient" value="0.000001" /> <!-- N/A -->
+  <xacro:property name="camera_yaw" value="0.000001" />
   <!-- Property Blocks -->
   <xacro:property name="body_inertia">
-    <inertia ixx="0.017" ixy="0.0" ixz="0.0" iyy="0.018" iyz="0.0" izz="0.028" /> <!-- [kg m^2] [kg m^2] [kg m^2] [kg m^2] [kg m^2] [kg m^2] -->
+    <inertia ixx="0.01" ixy="0.0" ixz="0.0" iyy="0.01" iyz="0.0" izz="0.01" /> <!-- [kg m^2] [kg m^2] [kg m^2] [kg m^2] [kg m^2] [kg m^2] -->
   </xacro:property>
   <!-- inertia of a single rotor, assuming it is a cuboid. Height=3mm, width=15mm -->
@@ -46,5 +52,5 @@
   </xacro:property>
   <!-- Included URDF Files -->
-  <xacro:include filename="$(find rotors_description)/urdf/multirotor_base.xacro" />
+  <xacro:include filename="$(find rotors_description)/urdf/multirotor_base_sphere.xacro" />
   <!-- Instantiate multirotor_base_macro once -->
   <xacro:multirotor_base_macro
@@ -74,8 +80,30 @@
     rotor_drag_coefficient="${rotor_drag_coefficient}"
     rolling_moment_coefficient="${rolling_moment_coefficient}"
-    color="Purple"
+    color="Red"
     use_own_mesh="false"
     mesh="">
     <origin xyz="${sqrt2inv * arm_length} -${sqrt2inv * arm_length} ${rotor_offset_top}" rpy="0 0 0" />
+    <!-- <origin xyz="0.07 -0.075 ${rotor_offset_top}" rpy="0 0 0" /> -->
+    <xacro:insert_block name="rotor_inertia" />
+  </xacro:vertical_rotor>
+  <xacro:vertical_rotor robot_namespace="${namespace}"
+    suffix="front_left"
+    direction="cw"
+    motor_constant="${motor_constant}"
+    moment_constant="${moment_constant}"
+    parent="${namespace}/base_link"
+    mass_rotor="${mass_rotor}"
+    radius_rotor="${radius_rotor}"
+    time_constant_up="${time_constant_up}"
+    time_constant_down="${time_constant_down}"
+    max_rot_velocity="${max_rot_velocity}"
+    motor_number="2"
+    rotor_drag_coefficient="${rotor_drag_coefficient}"
+    rolling_moment_coefficient="${rolling_moment_coefficient}"
+    color="Red"
+    use_own_mesh="false"
+    mesh="">
+    <origin xyz="${sqrt2inv * arm_length} ${sqrt2inv * arm_length} ${rotor_offset_top}" rpy="0 0 0" />
+    <!-- <origin xyz="0.07 0.075 ${rotor_offset_top}" rpy="0 0 0" /> -->
     <xacro:insert_block name="rotor_inertia" />
   </xacro:vertical_rotor>
@@ -95,28 +123,9 @@
     rotor_drag_coefficient="${rotor_drag_coefficient}"
     rolling_moment_coefficient="${rolling_moment_coefficient}"
-    color="Green"
+    color="Blue"
     use_own_mesh="false"
     mesh="">
     <origin xyz="-${sqrt2inv * arm_length} ${sqrt2inv * arm_length} ${rotor_offset_top}" rpy="0 0 0" />
-    <xacro:insert_block name="rotor_inertia" />
-  </xacro:vertical_rotor>
-  <xacro:vertical_rotor robot_namespace="${namespace}"
-    suffix="front_left"
-    direction="cw"
-    motor_constant="${motor_constant}"
-    moment_constant="${moment_constant}"
-    parent="${namespace}/base_link"
-    mass_rotor="${mass_rotor}"
-    radius_rotor="${radius_rotor}"
-    time_constant_up="${time_constant_up}"
-    time_constant_down="${time_constant_down}"
-    max_rot_velocity="${max_rot_velocity}"
-    motor_number="2"
-    rotor_drag_coefficient="${rotor_drag_coefficient}"
-    rolling_moment_coefficient="${rolling_moment_coefficient}"
-    color="Purple"
-    use_own_mesh="false"
-    mesh="">
-    <origin xyz="${sqrt2inv * arm_length} ${sqrt2inv * arm_length} ${rotor_offset_top}" rpy="0 0 0" />
+    <!-- <origin xyz="-0.07 0.075 ${rotor_offset_top}" rpy="0 0 0" /> -->
     <xacro:insert_block name="rotor_inertia" />
   </xacro:vertical_rotor>
@@ -135,8 +144,9 @@
     rotor_drag_coefficient="${rotor_drag_coefficient}"
     rolling_moment_coefficient="${rolling_moment_coefficient}"
-    color="Green"
+    color="Blue"
     use_own_mesh="false"
     mesh="">
     <origin xyz="-${sqrt2inv * arm_length} -${sqrt2inv * arm_length} ${rotor_offset_top}" rpy="0 0 0" />
+    <!-- <origin xyz="-0.07 -0.075 ${rotor_offset_top}" rpy="0 0 0" /> -->
     <xacro:insert_block name="rotor_inertia" />
   </xacro:vertical_rotor>

File: rotors_description/urdf/elios_VLP16_base.xacro (robot description, xacro)
@@ -39,7 +39,14 @@
   </xacro:if>
   <!-- Os1-64 -->
-  <xacro:include filename="$(find lidar_description)/urdf/OS1-64.urdf.xacro"/>
+  <!-- <xacro:include filename="$(find lidar_description)/urdf/OS1-64.urdf.xacro"/>
   <OS1-64 parent="${namespace}/base_link" name="${namespace}/os1" topic="/os1_points" hz="10" samples="100">
     <origin xyz="0 0 -0.07" rpy="3.14 0.0 3.14" />
-  </OS1-64>
+  </OS1-64> -->
+  <!-- VLP16 -->
+  <xacro:arg name="gpu" default="false"/>
+  <xacro:property name="gpu" value="$(arg gpu)" />
+  <xacro:include filename="$(find velodyne_description)/urdf/VLP-16.urdf.xacro"/>
+  <VLP-16 parent="${namespace}/base_link" name="/velodyne" topic="/velodyne_points" hz="10" samples="440" gpu="${gpu}">
+    <origin xyz="0 0 0.04" rpy="0 0 0" />
+  </VLP-16>
 </robot>
