Commit message: Separate model for m100 with odometry sensor

File: rotors_description/urdf/m100_base.xacro (robot description, xacro)
@@ -51,6 +51,14 @@
   <xacro:property name="gpu" value="$(arg gpu)" />
   <xacro:include filename="$(find lidar_description)/urdf/VLP-16.urdf.xacro"/>
-  <xacro:VLP-16 parent="${namespace}/base_link" name="${namespace}/velodyne" topic="velodyne_points" hz="10" samples="440" gpu="${gpu}">
+  <xacro:VLP-16 parent="${namespace}/base_link" name="${namespace}/velodyne" topic="velodyne_points" hz="10" samples="440" gpu="$(arg gpu)" collision_range="0.8">
     <origin xyz="0 0 0.04" rpy="0 0 0" />
   </xacro:VLP-16>
+  <!-- <xacro:include filename="$(find velodyne_description)/urdf/VLP-16.urdf.xacro"/>
+  <xacro:VLP-16 parent="base_link" name="velodyne" topic="velodyne_points" hz="10" samples="440" gpu="${gpu}">
+    <origin xyz="0 0 0.4" rpy="0 0 0" />
+  </xacro:VLP-16> -->
+  <!-- <xacro:include filename="$(find lidar_description)/urdf/OS0-128.urdf.xacro"/>
+  <xacro:OS0-128 parent="${namespace}/base_link" name="${namespace}/velodyne" topic="velodyne_points" hz="10" lasers="32" samples="440" collision_range="0.8" min_range="0.8">
+    <origin xyz="0 0 0.04" rpy="0 0 0" />
+  </xacro:OS0-128> -->
 </robot>
